Commit message: Sensor Lidar

File: scout_description/urdf/scout_mini.xacro (robot description, xacro)
@@ -140,8 +140,126 @@
         <axis xyz="0 0 1" rpy="0 0 0" />
     </joint>
-    <!-- Scout gazebo plugin -->
+<!-- Lidar Sensor -->
+    <xacro:property name="M_PI" value="3.1415926535897931" />
+    <xacro:macro name="lidar_sensor" params="
+        prefix:=''
+        parent:='base_link'
+        frame_id:='laser_frame'
+        xyz_offset:='0 0 0.0825'
+        rpy_offset:='0 0 0'
+        mesh_xyz_offset:='0 0 0'
+        mesh_rpy_offset:='${-M_PI/2} 0 0'
+        mesh_scale:='0.001 0.001 0.001'
+        collision_xyz_offset:='0 0 0'
+        collision_rpy_offset:='0 0 0'
+        inertial_xyz_offset:='0 0 0'
+        inertial_rpy_offset:='0 0 0'
+        lidar_width:=0.077
+        lidar_height:=0.0398
+        mass:=0.185
+        material_name:='rplidar_black'
+        material_color:='0.1 0.1 0.1 1'
+        gazebo_material_ambient:='0.1 0.1 0.1 1'
+        gazebo_material_diffuse:='0.1 0.1 0.1 1'
+        gazebo_material_specular:='0.1 0.1 0.1 1'
+        update_rate:=10
+        ray_count:=720
+        min_angle:='-3.14159'
+        max_angle:='3.14159'
+        min_range:='0.20'
+        max_range:='30.0'
+        range_resolution:='0.013'
+        topic_name:='scan'
+        always_on:=true
+        visualize:=false
+        enable_collision:=false">
+        <xacro:property name="radius" value="${lidar_width/2}" />
+        <xacro:property name="ixx_iyy" value="${(mass/12) * (3 * radius * radius + lidar_height * lidar_height)}" />
+        <xacro:property name="izz" value="${(mass/2) * (radius * radius)}" />
+        <link name="${prefix}${frame_id}">
+        <visual>
+            <origin xyz="${mesh_xyz_offset}" rpy="${mesh_rpy_offset}"/>
+            <geometry>
+            <mesh filename="package://scout_description/meshes/rplidar_s2.stl" scale="${mesh_scale}"/>
+            </geometry>
+            <material name="${material_name}">
+            <color rgba="${material_color}"/>
+            </material>
+        </visual>
+        <xacro:if value="${enable_collision}">
+            <collision>
+            <origin xyz="${collision_xyz_offset}" rpy="${collision_rpy_offset}"/>
+            <geometry>
+                <cylinder radius="${lidar_width/2}" length="${lidar_height}"/>
+            </geometry>
+            </collision>
+        </xacro:if>
+        <inertial>
+            <mass value="${mass}" />
+            <origin xyz="${inertial_xyz_offset}" rpy="${inertial_rpy_offset}"/>
+            <inertia
+            ixx="${ixx_iyy}"
+            ixy="0.0"
+            ixz="0.0"
+            iyy="${ixx_iyy}"
+            iyz="0.0"
+            izz="${izz}" />
+        </inertial>
+        </link>
+        <joint name="${prefix}${frame_id}_joint" type="fixed">
+        <parent link="${prefix}${parent}"/>
+        <child link="${prefix}${frame_id}" />
+        <origin xyz="${xyz_offset}" rpy="${rpy_offset}"/>
+        </joint>
+        <gazebo reference="${prefix}${frame_id}">
+        <material>
+            <ambient>${gazebo_material_ambient}</ambient>
+            <diffuse>${gazebo_material_diffuse}</diffuse>
+            <specular>${gazebo_material_specular}</specular>
+        </material>
+        <sensor name="${prefix}lidar_sensor" type="gpu_lidar">
+            <topic>${topic_name}</topic>
+            <update_rate>${update_rate}</update_rate>
+            <always_on>${always_on}</always_on>
+            <visualize>${visualize}</visualize>
+            <ray>
+            <scan>
+                <horizontal>
+                <samples>${ray_count}</samples>
+                <resolution>1</resolution>
+                <min_angle>${min_angle}</min_angle>
+                <max_angle>${max_angle}</max_angle>
+                </horizontal>
+                <vertical>
+                <samples>1</samples>
+                <resolution>1</resolution>
+                <min_angle>0</min_angle>
+                <max_angle>0</max_angle>
+                </vertical>
+            </scan>
+            <range>
+                <min>${min_range}</min>
+                <max>${max_range}</max>
+                <resolution>${range_resolution}</resolution>
+            </range>
+            </ray>
+            <gz_frame_id>${prefix}${frame_id}</gz_frame_id>
+        </sensor>
+        </gazebo>
+    </xacro:macro>
+    <xacro:arg name="prefix" default=""/>
+    <xacro:lidar_sensor
+    prefix="$(arg prefix)"
+    parent="base_link"
+    frame_id="laser_frame"
+    xyz_offset="0 0 0.0825"
+    rpy_offset="0 0 3.14"
+    mesh_xyz_offset="0 0 0"
+    mesh_rpy_offset="${-M_PI/2} 0 0"
+    topic_name="scan"/>
+<!-- Scout gazebo plugin -->
     <gazebo>
-        <plugin filename="libignition-gazebo-joint-state-publisher-system.so"
-            name="ignition::gazebo::systems::JointStatePublisher">
+        <plugin filename="libgz-sim-joint-state-publisher-system.so"
+            name="gz::sim::systems::JointStatePublisher">
             <topic>joint_states</topic>
             <update_rate>50</update_rate>
@@ -152,6 +270,6 @@
         </plugin>
         <plugin
-            filename="libignition-gazebo-diff-drive-system.so"
-            name="ignition::gazebo::systems::DiffDrive">
+            filename="libgz-sim-diff-drive-system.so"
+            name="gz::sim::systems::DiffDrive">
             <left_joint>front_left_wheel</left_joint>
             <right_joint>front_right_wheel</right_joint>

Commit message: camera RGB

File: scout_description/urdf/scout_mini.xacro (robot description, xacro)
@@ -258,4 +258,75 @@
     mesh_rpy_offset="${-M_PI/2} 0 0"
     topic_name="scout_mini/scan"/>
+      <!-- 7 - Camera -->
+  <joint type="fixed" name="camera_joint">
+    <origin xyz="0.225 0 0.075" rpy="0 0 0"/>
+    <child link="camera_link"/>
+    <parent link="base_link"/>
+    <axis xyz="0 1 0" />
+  </joint>
+  <link name='camera_link'>
+    <pose>0 0 0 0 0 0</pose>
+    <inertial>
+      <mass value="0.1"/>
+      <origin xyz="0 0 0" rpy="0 0 0"/>
+      <inertia
+          ixx="1e-6" ixy="0" ixz="0"
+          iyy="1e-6" iyz="0"
+          izz="1e-6" />
+    </inertial>
+    <collision name='collision'>
+      <origin xyz="0 0 0" rpy="0 0 0"/>
+      <geometry>
+        <box size=".03 .03 .03"/>
+      </geometry>
+    </collision>
+    <visual name='camera_link_visual'>
+      <origin xyz="0 0 0" rpy="0 0 0"/>
+      <geometry>
+        <box size=".03 .03 .03"/>
+      </geometry>
+    </visual>
+  </link>
+  <gazebo reference="camera_link">
+    <material>Gazebo/Red</material>
+  </gazebo>
+  <joint type="fixed" name="camera_optical_joint">
+    <origin xyz="0 0 0" rpy="-1.5707 0 -1.5707"/>
+    <child link="camera_link_optical"/>
+    <parent link="camera_link"/>
+  </joint>
+  <link name="camera_link_optical">
+  </link>
+    <!-- 7 - Camera Gazebo Plugin -->
+  <gazebo reference="camera_link">
+    <sensor name="camera" type="camera">
+      <camera>
+        <horizontal_fov>1.3962634</horizontal_fov>
+        <image>
+          <width>640</width>
+          <height>480</height>
+          <format>R8G8B8</format>
+        </image>
+        <clip>
+          <near>0.1</near>
+          <far>15</far>
+        </clip>
+        <noise>
+          <type>gaussian</type>
+          <!-- Noise is sampled independently per pixel on each frame.
+               That pixel's noise value is added to each of its color
+               channels, which at that point lie in the range [0,1]. -->
+          <mean>0.0</mean>
+          <stddev>0.007</stddev>
+        </noise>
+        <optical_frame_id>camera_link_optical</optical_frame_id>
+        <camera_info_topic>scout_mini/rgb_cam/camera_info</camera_info_topic>
+      </camera>
+      <always_on>1</always_on>
+      <update_rate>20</update_rate>
+      <visualize>true</visualize>
+      <topic>scout_mini/rgb_cam/image</topic>
+    </sensor>
+  </gazebo>
 <!-- Scout gazebo plugin -->
     <gazebo>

Commit message: verlab

File: scout_description/urdf/scout_mini.xacro (robot description, xacro)
@@ -281,14 +281,14 @@
       </geometry>
     </collision>
-    <visual name='camera_link_visual'>
-      <origin xyz="0 0 0" rpy="0 0 0"/>
-      <geometry>
-        <box size=".03 .03 .03"/>
-      </geometry>
-    </visual>
+    <visual>
+        <origin xyz="0 0 0" rpy="${M_PI/2} 0.0 ${M_PI/2}"/>
+        <geometry>
+          <mesh filename="package://scout_description/meshes/d435.stl" />
+        </geometry>
+        <material name="aluminum">
+          <color rgba="0.8 0.8 0.8 1"/>
+        </material>
+      </visual>
   </link>
-  <gazebo reference="camera_link">
-    <material>Gazebo/Red</material>
-  </gazebo>
   <joint type="fixed" name="camera_optical_joint">
     <origin xyz="0 0 0" rpy="-1.5707 0 -1.5707"/>

Commit message: organização do codigo

File: scout_description/urdf/scout_mini.xacro (robot description, xacro)
@@ -140,5 +140,5 @@
         <axis xyz="0 0 1" rpy="0 0 0" />
     </joint>
-<!-- Lidar Sensor -->
+    <!-- Lidar Sensor -->
     <xacro:property name="M_PI" value="3.1415926535897931" />
     <xacro:macro name="lidar_sensor" params="
@@ -208,42 +208,42 @@
         </link>
         <joint name="${prefix}${frame_id}_joint" type="fixed">
-        <parent link="${prefix}${parent}"/>
-        <child link="${prefix}${frame_id}" />
-        <origin xyz="${xyz_offset}" rpy="${rpy_offset}"/>
+            <parent link="${prefix}${parent}"/>
+            <child link="${prefix}${frame_id}" />
+            <origin xyz="${xyz_offset}" rpy="${rpy_offset}"/>
         </joint>
         <gazebo reference="${prefix}${frame_id}">
-        <material>
-            <ambient>${gazebo_material_ambient}</ambient>
-            <diffuse>${gazebo_material_diffuse}</diffuse>
-            <specular>${gazebo_material_specular}</specular>
-        </material>
-        <sensor name="${prefix}lidar_sensor" type="gpu_lidar">
-            <topic>${topic_name}</topic>
-            <update_rate>${update_rate}</update_rate>
-            <always_on>${always_on}</always_on>
-            <visualize>${visualize}</visualize>
-            <ray>
-            <scan>
-                <horizontal>
-                <samples>${ray_count}</samples>
-                <resolution>1</resolution>
-                <min_angle>${min_angle}</min_angle>
-                <max_angle>${max_angle}</max_angle>
-                </horizontal>
-                <vertical>
-                <samples>1</samples>
-                <resolution>1</resolution>
-                <min_angle>0</min_angle>
-                <max_angle>0</max_angle>
-                </vertical>
-            </scan>
-            <range>
-                <min>${min_range}</min>
-                <max>${max_range}</max>
-                <resolution>${range_resolution}</resolution>
-            </range>
-            </ray>
-            <gz_frame_id>${prefix}${frame_id}</gz_frame_id>
-        </sensor>
+            <material>
+                <ambient>${gazebo_material_ambient}</ambient>
+                <diffuse>${gazebo_material_diffuse}</diffuse>
+                <specular>${gazebo_material_specular}</specular>
+            </material>
+            <sensor name="${prefix}lidar_sensor" type="gpu_lidar">
+                <topic>${topic_name}</topic>
+                <update_rate>${update_rate}</update_rate>
+                <always_on>${always_on}</always_on>
+                <visualize>${visualize}</visualize>
+                <ray>
+                <scan>
+                    <horizontal>
+                    <samples>${ray_count}</samples>
+                    <resolution>1</resolution>
+                    <min_angle>${min_angle}</min_angle>
+                    <max_angle>${max_angle}</max_angle>
+                    </horizontal>
+                    <vertical>
+                    <samples>1</samples>
+                    <resolution>1</resolution>
+                    <min_angle>0</min_angle>
+                    <max_angle>0</max_angle>
+                    </vertical>
+                </scan>
+                <range>
+                    <min>${min_range}</min>
+                    <max>${max_range}</max>
+                    <resolution>${range_resolution}</resolution>
+                </range>
+                </ray>
+                <gz_frame_id>${prefix}${frame_id}</gz_frame_id>
+            </sensor>
         </gazebo>
     </xacro:macro>
@@ -258,76 +258,76 @@
     mesh_rpy_offset="${-M_PI/2} 0 0"
     topic_name="scout_mini/scan"/>
-      <!-- 7 - Camera -->
-  <joint type="fixed" name="camera_joint">
-    <origin xyz="0.225 0 0.075" rpy="0 0 0"/>
-    <child link="camera_link"/>
-    <parent link="base_link"/>
-    <axis xyz="0 1 0" />
-  </joint>
-  <link name='camera_link'>
-    <pose>0 0 0 0 0 0</pose>
-    <inertial>
-      <mass value="0.1"/>
-      <origin xyz="0 0 0" rpy="0 0 0"/>
-      <inertia
-          ixx="1e-6" ixy="0" ixz="0"
-          iyy="1e-6" iyz="0"
-          izz="1e-6" />
-    </inertial>
-    <collision name='collision'>
-      <origin xyz="0 0 0" rpy="0 0 0"/>
-      <geometry>
-        <box size=".03 .03 .03"/>
-      </geometry>
-    </collision>
-    <visual>
-        <origin xyz="0 0 0" rpy="${M_PI/2} 0.0 ${M_PI/2}"/>
-        <geometry>
-          <mesh filename="package://scout_description/meshes/d435.stl" />
-        </geometry>
-        <material name="aluminum">
-          <color rgba="0.8 0.8 0.8 1"/>
-        </material>
-      </visual>
-  </link>
-  <joint type="fixed" name="camera_optical_joint">
-    <origin xyz="0 0 0" rpy="-1.5707 0 -1.5707"/>
-    <child link="camera_link_optical"/>
-    <parent link="camera_link"/>
-  </joint>
-  <link name="camera_link_optical">
-  </link>
+    <!-- Camera -->
+    <joint type="fixed" name="camera_joint">
+        <origin xyz="0.225 0 0.075" rpy="0 0 0"/>
+        <child link="camera_link"/>
+        <parent link="base_link"/>
+        <axis xyz="0 1 0" />
+    </joint>
+    <link name='camera_link'>
+        <pose>0 0 0 0 0 0</pose>
+        <inertial>
+        <mass value="0.1"/>
+        <origin xyz="0 0 0" rpy="0 0 0"/>
+        <inertia
+            ixx="1e-6" ixy="0" ixz="0"
+            iyy="1e-6" iyz="0"
+            izz="1e-6" />
+        </inertial>
+        <collision name='collision'>
+            <origin xyz="0 0 0" rpy="0 0 0"/>
+            <geometry>
+                <box size=".03 .03 .03"/>
+            </geometry>
+        </collision>
+        <visual>
+            <origin xyz="0 0 0" rpy="${M_PI/2} 0.0 ${M_PI/2}"/>
+            <geometry>
+                <mesh filename="package://scout_description/meshes/d435.stl"/>
+            </geometry>
+            <material name="aluminum">
+            <color rgba="0.8 0.8 0.8 1"/>
+            </material>
+        </visual>
+    </link>
+    <joint type="fixed" name="camera_optical_joint">
+        <origin xyz="0 0 0" rpy="-1.5707 0 -1.5707"/>
+        <child link="camera_link_optical"/>
+        <parent link="camera_link"/>
+    </joint>
+    <link name="camera_link_optical">
+    </link>
     <!-- 7 - Camera Gazebo Plugin -->
-  <gazebo reference="camera_link">
-    <sensor name="camera" type="camera">
-      <camera>
-        <horizontal_fov>1.3962634</horizontal_fov>
-        <image>
-          <width>640</width>
-          <height>480</height>
-          <format>R8G8B8</format>
-        </image>
-        <clip>
-          <near>0.1</near>
-          <far>15</far>
-        </clip>
-        <noise>
-          <type>gaussian</type>
-          <!-- Noise is sampled independently per pixel on each frame.
-               That pixel's noise value is added to each of its color
-               channels, which at that point lie in the range [0,1]. -->
-          <mean>0.0</mean>
-          <stddev>0.007</stddev>
-        </noise>
-        <optical_frame_id>camera_link_optical</optical_frame_id>
-        <camera_info_topic>scout_mini/rgb_cam/camera_info</camera_info_topic>
-      </camera>
-      <always_on>1</always_on>
-      <update_rate>20</update_rate>
-      <visualize>true</visualize>
-      <topic>scout_mini/rgb_cam/image</topic>
-    </sensor>
-  </gazebo>
-<!-- Scout gazebo plugin -->
+    <gazebo reference="camera_link">
+        <sensor name="camera" type="camera">
+            <camera>
+                <horizontal_fov>1.3962634</horizontal_fov>
+                <image>
+                    <width>640</width>
+                    <height>480</height>
+                    <format>R8G8B8</format>
+                </image>
+                <clip>
+                    <near>0.1</near>
+                    <far>15</far>
+                </clip>
+                <noise>
+                    <type>gaussian</type>
+                    <!-- Noise is sampled independently per pixel on each frame.
+                        That pixel's noise value is added to each of its color
+                        channels, which at that point lie in the range [0,1]. -->
+                    <mean>0.0</mean>
+                    <stddev>0.007</stddev>
+                </noise>
+                <optical_frame_id>camera_link_optical</optical_frame_id>
+                <camera_info_topic>scout_mini/rgb_cam/camera_info</camera_info_topic>
+            </camera>
+            <always_on>1</always_on>
+            <update_rate>20</update_rate>
+            <visualize>true</visualize>
+            <topic>scout_mini/rgb_cam/image</topic>
+        </sensor>
+    </gazebo>
+    <!-- Scout gazebo plugin -->
     <gazebo>
         <plugin filename="libgz-sim-joint-state-publisher-system.so"
