Commit message: modularização e novos sensores

File: scout_description/urdf/scout_mini.xacro (robot description, xacro)
@@ -1,254 +1,17 @@
 <?xml version="1.0"?>
 <robot name="scout_mini" xmlns:xacro="http://ros.org/wiki/xacro">
-    <!-- Vehicle Geometries -->
-    <!-- Base link -->
-    <link name="base_link">
-        <visual>
-            <origin xyz="0 0 0" rpy="1.57 0 -1.57" />
-            <geometry>
-                <mesh
-                    filename="package://scout_description/meshes/scout_mini_base_link.dae" />
-            </geometry>
-        </visual>
-        <collision>
-            <origin xyz="0 0 0" rpy="1.57 0 -1.57" />
-            <geometry>
-                <mesh
-                    filename="package://scout_description/meshes/scout_mini_base_link.dae" />
-            </geometry>
-        </collision>
-    </link>
-    <link
-        name="inertial_link">
-        <inertial>
-            <mass value="132.3898489950015" />
-            <origin xyz=" 0 0 0" />
-            <inertia ixx="0.185196122711036" ixy="4.30144213829512E-08" ixz="5.81037523686401E-08"
-                iyy="0.364893736238929" iyz="-0.000386720198091934" izz="0.223868521722778" />
-        </inertial>
-    </link>
-    <joint
-        name="inertial_joint" type="fixed">
-        <origin xyz="0 0 0" rpy="0 0 0" />
-        <parent link="base_link" />
-        <child link="inertial_link" />
-    </joint>
-    <!-- Scout wheel -->
-    <link
-        name="front_right_wheel_link">
-        <inertial>
-            <mass value="3" />
-            <origin xyz="0 0 0" />
-            <inertia ixx="0.7171" ixy="0" ixz="0" iyy="0.7171" iyz="0" izz="0.1361" />
-        </inertial>
-        <visual>
-            <origin xyz="0 0 0" rpy="0 0 0" />
-            <geometry>
-                <mesh filename="package://scout_description/meshes/wheel.dae" />
-            </geometry>
-        </visual>
-        <collision>
-            <origin xyz="0 0 0" rpy="0 0 0" />
-            <geometry>
-                <mesh filename="package://scout_description/meshes/wheel.dae" />
-            </geometry>
-        </collision>
-    </link>
-    <joint
-        name="front_right_wheel" type="continuous">
-        <origin rpy="1.57 0 0" xyz="0.2319755 -0.2082515 -0.099998" />
-        <parent link="base_link" />
-        <child link="front_right_wheel_link" />
-        <axis xyz="0 0 -1" rpy="0 0 0" />
-    </joint>
-    <link name="front_left_wheel_link">
-        <inertial>
-            <mass value="3" />
-            <origin xyz="0 0 0" />
-            <inertia ixx="0.7171" ixy="0" ixz="0" iyy="0.7171" iyz="0" izz="0.1361" />
-        </inertial>
-        <visual>
-            <origin xyz="0 0 0" rpy="0 0 0" />
-            <geometry>
-                <mesh filename="package://scout_description/meshes/wheel.dae" />
-            </geometry>
-        </visual>
-        <collision>
-            <origin xyz="0 0 0" rpy="0 0 0" />
-            <geometry>
-                <mesh filename="package://scout_description/meshes/wheel.dae" />
-            </geometry>
-        </collision>
-    </link>
-    <joint
-        name="front_left_wheel" type="continuous">
-        <origin rpy="-1.57 0 0" xyz="0.2319755 0.2082515 -0.100998" />
-        <parent link="base_link" />
-        <child link="front_left_wheel_link" />
-        <axis xyz="0 0 1" rpy="0 0 0" />
-    </joint>
-    <link name="rear_right_wheel_link">
-        <inertial>
-            <mass value="3" />
-            <origin xyz="0 0 0" />
-            <inertia ixx="0.7171" ixy="0" ixz="0" iyy="0.7171" iyz="0" izz="0.1361" />
-        </inertial>
-        <visual>
-            <origin xyz="0 0 0" rpy="0 0 0" />
-            <geometry>
-                <mesh filename="package://scout_description/meshes/wheel.dae" />
-            </geometry>
-        </visual>
-        <collision>
-            <origin xyz="0 0 0" rpy="0 0 0" />
-            <geometry>
-                <mesh filename="package://scout_description/meshes/wheel.dae" />
-            </geometry>
-        </collision>
-    </link>
-    <joint
-        name="rear_right_wheel" type="continuous">
-        <origin rpy="1.57 0 0" xyz="-0.2319755 -0.2082515 -0.099998" />
-        <parent link="base_link" />
-        <child link="rear_right_wheel_link" />
-        <axis xyz="0 0 -1" rpy="0 0 0" />
-    </joint>
-    <link name="rear_left_wheel_link">
-        <inertial>
-            <mass value="3" />
-            <origin xyz="0 0 0" />
-            <inertia ixx="0.7171" ixy="0" ixz="0" iyy="0.7171" iyz="0" izz="0.1361" />
-        </inertial>
-        <visual>
-            <origin xyz="0 0 0" rpy="0 0 0" />
-            <geometry>
-                <mesh filename="package://scout_description/meshes/wheel.dae" />
-            </geometry>
-        </visual>
-        <collision>
-            <origin xyz="0 0 0" rpy="0 0 0" />
-            <geometry>
-                <mesh filename="package://scout_description/meshes/wheel.dae" />
-            </geometry>
-        </collision>
-    </link>
-    <joint
-        name="rear_left_wheel" type="continuous">
-        <origin rpy="-1.57 0 0" xyz="-0.2319755 0.2082515 -0.100998" />
-        <parent link="base_link" />
-        <child link="rear_left_wheel_link" />
-        <axis xyz="0 0 1" rpy="0 0 0" />
-    </joint>
+    <xacro:property name="M_PI" value="3.1415926535897931" />
+    <xacro:include filename="$(find scout_description)/urdf/mech/scout_mini_base.xacro"/>
+    <xacro:include filename="$(find scout_description)/urdf/mech/scout_mini_wheels.xacro"/>
+    <xacro:include filename="$(find scout_description)/urdf/sensors/lidar.xacro"/>
+    <xacro:include filename="$(find scout_description)/urdf/sensors/lidar3d.xacro"/>
+    <xacro:include filename="$(find scout_description)/urdf/sensors/camera.xacro"/>
+    <xacro:include filename="$(find scout_description)/urdf/sensors/RGBcamera.xacro"/>
+    <!-- Robot -->
+    <xacro:scout_mini_base/>
+    <xacro:scout_mini_wheels/>
+    <!-- Sensors -->
     <!-- Lidar Sensor -->
-    <xacro:property name="M_PI" value="3.1415926535897931" />
-    <xacro:macro name="lidar_sensor" params="
-        prefix:=''
-        parent:='base_link'
-        frame_id:='laser_frame'
-        xyz_offset:='0 0 0.0825'
-        rpy_offset:='0 0 0'
-        mesh_xyz_offset:='0 0 0'
-        mesh_rpy_offset:='${-M_PI/2} 0 0'
-        mesh_scale:='0.001 0.001 0.001'
-        collision_xyz_offset:='0 0 0'
-        collision_rpy_offset:='0 0 0'
-        inertial_xyz_offset:='0 0 0'
-        inertial_rpy_offset:='0 0 0'
-        lidar_width:=0.077
-        lidar_height:=0.0398
-        mass:=0.185
-        material_name:='rplidar_black'
-        material_color:='0.1 0.1 0.1 1'
-        gazebo_material_ambient:='0.1 0.1 0.1 1'
-        gazebo_material_diffuse:='0.1 0.1 0.1 1'
-        gazebo_material_specular:='0.1 0.1 0.1 1'
-        update_rate:=10
-        ray_count:=720
-        min_angle:='-3.14159'
-        max_angle:='3.14159'
-        min_range:='0.20'
-        max_range:='30.0'
-        range_resolution:='0.013'
-        topic_name:='scout_mini/scan'
-        always_on:=true
-        visualize:=false
-        enable_collision:=false">
-        <xacro:property name="radius" value="${lidar_width/2}" />
-        <xacro:property name="ixx_iyy" value="${(mass/12) * (3 * radius * radius + lidar_height * lidar_height)}" />
-        <xacro:property name="izz" value="${(mass/2) * (radius * radius)}" />
-        <link name="${prefix}${frame_id}">
-        <visual>
-            <origin xyz="${mesh_xyz_offset}" rpy="${mesh_rpy_offset}"/>
-            <geometry>
-            <mesh filename="package://scout_description/meshes/rplidar_s2.stl" scale="${mesh_scale}"/>
-            </geometry>
-            <material name="${material_name}">
-            <color rgba="${material_color}"/>
-            </material>
-        </visual>
-        <xacro:if value="${enable_collision}">
-            <collision>
-            <origin xyz="${collision_xyz_offset}" rpy="${collision_rpy_offset}"/>
-            <geometry>
-                <cylinder radius="${lidar_width/2}" length="${lidar_height}"/>
-            </geometry>
-            </collision>
-        </xacro:if>
-        <inertial>
-            <mass value="${mass}" />
-            <origin xyz="${inertial_xyz_offset}" rpy="${inertial_rpy_offset}"/>
-            <inertia
-            ixx="${ixx_iyy}"
-            ixy="0.0"
-            ixz="0.0"
-            iyy="${ixx_iyy}"
-            iyz="0.0"
-            izz="${izz}" />
-        </inertial>
-        </link>
-        <joint name="${prefix}${frame_id}_joint" type="fixed">
-            <parent link="${prefix}${parent}"/>
-            <child link="${prefix}${frame_id}" />
-            <origin xyz="${xyz_offset}" rpy="${rpy_offset}"/>
-        </joint>
-        <gazebo reference="${prefix}${frame_id}">
-            <material>
-                <ambient>${gazebo_material_ambient}</ambient>
-                <diffuse>${gazebo_material_diffuse}</diffuse>
-                <specular>${gazebo_material_specular}</specular>
-            </material>
-            <sensor name="${prefix}lidar_sensor" type="gpu_lidar">
-                <topic>${topic_name}</topic>
-                <update_rate>${update_rate}</update_rate>
-                <always_on>${always_on}</always_on>
-                <visualize>${visualize}</visualize>
-                <ray>
-                <scan>
-                    <horizontal>
-                    <samples>${ray_count}</samples>
-                    <resolution>1</resolution>
-                    <min_angle>${min_angle}</min_angle>
-                    <max_angle>${max_angle}</max_angle>
-                    </horizontal>
-                    <vertical>
-                    <samples>1</samples>
-                    <resolution>1</resolution>
-                    <min_angle>0</min_angle>
-                    <max_angle>0</max_angle>
-                    </vertical>
-                </scan>
-                <range>
-                    <min>${min_range}</min>
-                    <max>${max_range}</max>
-                    <resolution>${range_resolution}</resolution>
-                </range>
-                </ray>
-                <gz_frame_id>${prefix}${frame_id}</gz_frame_id>
-            </sensor>
-        </gazebo>
-    </xacro:macro>
-    <xacro:arg name="prefix" default=""/>
-    <xacro:lidar_sensor
-    prefix="$(arg prefix)"
+    <xacro:lidar
     parent="base_link"
     frame_id="laser_frame"
@@ -258,75 +21,20 @@
     mesh_rpy_offset="${-M_PI/2} 0 0"
     topic_name="scout_mini/scan"/>
+    <!-- 3D Lidar Sensor -->
+    <xacro:lidar3d
+    parent="base_link"
+    frame_id="3dlaser_frame"
+    xyz_offset="0 0 0.0825"
+    rpy_offset="0 0 3.14"
+    mesh_xyz_offset="0 0 0"
+    mesh_rpy_offset="${-M_PI/2} 0 0"
+    topic_name="scout_mini/scan3d"/>
     <!-- Camera -->
-    <joint type="fixed" name="camera_joint">
-        <origin xyz="0.225 0 0.075" rpy="0 0 0"/>
-        <child link="camera_link"/>
-        <parent link="base_link"/>
-        <axis xyz="0 1 0" />
-    </joint>
-    <link name='camera_link'>
-        <pose>0 0 0 0 0 0</pose>
-        <inertial>
-        <mass value="0.1"/>
-        <origin xyz="0 0 0" rpy="0 0 0"/>
-        <inertia
-            ixx="1e-6" ixy="0" ixz="0"
-            iyy="1e-6" iyz="0"
-            izz="1e-6" />
-        </inertial>
-        <collision name='collision'>
-            <origin xyz="0 0 0" rpy="0 0 0"/>
-            <geometry>
-                <box size=".03 .03 .03"/>
-            </geometry>
-        </collision>
-        <visual>
-            <origin xyz="0 0 0" rpy="${M_PI/2} 0.0 ${M_PI/2}"/>
-            <geometry>
-                <mesh filename="package://scout_description/meshes/d435.stl"/>
-            </geometry>
-            <material name="aluminum">
-            <color rgba="0.8 0.8 0.8 1"/>
-            </material>
-        </visual>
-    </link>
-    <joint type="fixed" name="camera_optical_joint">
-        <origin xyz="0 0 0" rpy="-1.5707 0 -1.5707"/>
-        <child link="camera_link_optical"/>
-        <parent link="camera_link"/>
-    </joint>
-    <link name="camera_link_optical">
-    </link>
-    <!-- 7 - Camera Gazebo Plugin -->
-    <gazebo reference="camera_link">
-        <sensor name="camera" type="camera">
-            <camera>
-                <horizontal_fov>1.3962634</horizontal_fov>
-                <image>
-                    <width>640</width>
-                    <height>480</height>
-                    <format>R8G8B8</format>
-                </image>
-                <clip>
-                    <near>0.1</near>
-                    <far>15</far>
-                </clip>
-                <noise>
-                    <type>gaussian</type>
-                    <!-- Noise is sampled independently per pixel on each frame.
-                        That pixel's noise value is added to each of its color
-                        channels, which at that point lie in the range [0,1]. -->
-                    <mean>0.0</mean>
-                    <stddev>0.007</stddev>
-                </noise>
-                <optical_frame_id>camera_link_optical</optical_frame_id>
-                <camera_info_topic>scout_mini/rgb_cam/camera_info</camera_info_topic>
-            </camera>
-            <always_on>1</always_on>
-            <update_rate>20</update_rate>
-            <visualize>true</visualize>
-            <topic>scout_mini/rgb_cam/image</topic>
-        </sensor>
-    </gazebo>
+    <xacro:camera/>
+    <!--RGBD Camera -->
+    <xacro:RGBcamera
+    camera_name="RGBcamera"
+    xyz_offset="0.26 0 0"
+    rpy_offset="0 0 0"/>
     <!-- Scout gazebo plugin -->
     <gazebo>
