Commit message: finalizado

File: scout_description/urdf/mech/scout_mini_wheels.xacro (robot description, xacro)
@@ -12,5 +12,5 @@
                 <origin xyz="0 0 0" rpy="0 0 0" />
                 <geometry>
-                    <mesh filename="package://scout_description/meshes/wheel.dae" />
+                    <mesh filename="package://scout_description/meshes/scout_mini_wheel.dae" />
                 </geometry>
             </visual>
@@ -18,5 +18,5 @@
                 <origin xyz="0 0 0" rpy="0 0 0" />
                 <geometry>
-                    <mesh filename="package://scout_description/meshes/wheel.dae" />
+                    <mesh filename="package://scout_description/meshes/scout_mini_wheel.dae" />
                 </geometry>
             </collision>
@@ -38,5 +38,5 @@
                 <origin xyz="0 0 0" rpy="0 0 0" />
                 <geometry>
-                    <mesh filename="package://scout_description/meshes/wheel.dae" />
+                    <mesh filename="package://scout_description/meshes/scout_mini_wheel.dae" />
                 </geometry>
             </visual>
@@ -44,5 +44,5 @@
                 <origin xyz="0 0 0" rpy="0 0 0" />
                 <geometry>
-                    <mesh filename="package://scout_description/meshes/wheel.dae" />
+                    <mesh filename="package://scout_description/meshes/scout_mini_wheel.dae" />
                 </geometry>
             </collision>
@@ -64,5 +64,5 @@
                 <origin xyz="0 0 0" rpy="0 0 0" />
                 <geometry>
-                    <mesh filename="package://scout_description/meshes/wheel.dae" />
+                    <mesh filename="package://scout_description/meshes/scout_mini_wheel.dae" />
                 </geometry>
             </visual>
@@ -70,5 +70,5 @@
                 <origin xyz="0 0 0" rpy="0 0 0" />
                 <geometry>
-                    <mesh filename="package://scout_description/meshes/wheel.dae" />
+                    <mesh filename="package://scout_description/meshes/scout_mini_wheel.dae" />
                 </geometry>
             </collision>
@@ -90,5 +90,5 @@
                 <origin xyz="0 0 0" rpy="0 0 0" />
                 <geometry>
-                    <mesh filename="package://scout_description/meshes/wheel.dae" />
+                    <mesh filename="package://scout_description/meshes/scout_mini_wheel.dae" />
                 </geometry>
             </visual>
@@ -96,5 +96,5 @@
                 <origin xyz="0 0 0" rpy="0 0 0" />
                 <geometry>
-                    <mesh filename="package://scout_description/meshes/wheel.dae" />
+                    <mesh filename="package://scout_description/meshes/scout_mini_wheel.dae" />
                 </geometry>
             </collision>

File: scout_description/urdf/scout_mini.xacro (robot description, xacro)
@@ -13,28 +13,11 @@
     <!-- Sensors -->
     <!-- Lidar Sensor -->
-    <xacro:lidar
-    parent="base_link"
-    frame_id="laser_frame"
-    xyz_offset="0 0 0.0825"
-    rpy_offset="0 0 3.14"
-    mesh_xyz_offset="0 0 0"
-    mesh_rpy_offset="${-M_PI/2} 0 0"
-    topic_name="scout_mini/scan"/>
+    <xacro:lidar/>
     <!-- 3D Lidar Sensor -->
-    <xacro:lidar3d
-    parent="base_link"
-    frame_id="3dlaser_frame"
-    xyz_offset="0 0 0.0825"
-    rpy_offset="0 0 3.14"
-    mesh_xyz_offset="0 0 0"
-    mesh_rpy_offset="${-M_PI/2} 0 0"
-    topic_name="scout_mini/scan3d"/>
+    <xacro:lidar3d/>
     <!-- Camera -->
     <xacro:camera/>
     <!--RGBD Camera -->
-    <xacro:RGBcamera
-    camera_name="RGBcamera"
-    xyz_offset="0.26 0 0"
-    rpy_offset="0 0 0"/>
+    <xacro:RGBcamera/>
     <!-- Scout gazebo plugin -->
     <gazebo>

File: scout_description/urdf/sensors/RGBcamera.xacro (robot description, xacro)
@@ -6,6 +6,6 @@
     parent:='base_link'
     mesh_file:='package://scout_description/meshes/d435.stl'
-    xyz_offset:='0.105 0 0.05'
-    rpy_offset:='0 -0.50 0'
+    xyz_offset:='0.26 0 0'
+    rpy_offset:='0 0 0'
     mesh_xyz_offset:='0 0 0'
     mesh_rpy_offset:='${M_PI/2} 0.0 ${M_PI/2}'
